File: PCB/WizServoTester.kicad_sch (KiCad schematic)
At the start: 38 parts, among them J1 USB_C_Receptacle_USB2.0_16P, J2 Servo_3_Header, J3 Servo_4_Header, J4 Servo_1_Header, J5 Servo_2_Header, J6 BAT_XT60, J7 BAT_Powerpole, J8 BAT_Pads, SW1 EC 11, SW2 EC 11, SW3 EC 11, SW4 EC 11, SW5 SW_Push, SW6 SW_SPDT, SW7 SW_Push, U1 ESP32-C6-WROOM-1, U2 USBLC6-2SC6, U3 AMS1117-3.3, U4 Mini560

Commit message: Kicad Files
Parts:
- removed J7: BAT_Powerpole, Connector_AMASS:AMASS_XT30PW-M_1x02_P2.50mm_Horizontal, symbol Connector_Generic:Conn_01x02
- added H1, H2: M3 Mounting Hole, MountingHole:MountingHole_3.2mm_M3, symbol Mechanical:MountingHole
- C1, C2, C3, C4, C5, C6, C7, C9: footprint (none) -> Capacitor_SMD:C_0805_2012Metric
- C8: value 1000u 16v -> 470u 16v; footprint (none) -> Capacitor_SMD:CP_Elec_8x10.5
- D2, D4: footprint (none) -> Diode_SMD:D_SMA
- J1: footprint Connector_USB:USB_C_Plug_Molex_105444 -> Connector_USB:USB_C_Receptacle_HCTL_HC-TYPE-C-16P-01A
- J6: value BAT_XT60 -> BAT_XT30; footprint Connector_AMASS:AMASS_XT30PW-M_1x02_P2.50mm_Horizontal -> Connector_AMASS:AMASS_XT30U-F_1x02_P5.0mm_Vertical
- J8: footprint Connector_AMASS:AMASS_XT30PW-M_1x02_P2.50mm_Horizontal -> TestPoint:TestPoint_2Pads_Pitch5.08mm_Drill1.3mm
- R1, R4, R5, R6: footprint (none) -> Resistor_SMD:R_0805_2012Metric
- R2, R3: value 10k -> 5.1k; footprint (none) -> Resistor_SMD:R_0805_2012Metric
- SW1, SW2, SW3, SW4: footprint (none) -> Rotary_Encoder:RotaryEncoder_Alps_EC11E-Switch_Vertical_H20mm_MountingHoles
- SW5, SW7: footprint (none) -> Button_Switch_SMD:SW_SPST_TS-1088-xR020
- SW6: footprint (none) -> '${KICAD_3RD_PARTY}/EasyEDA.pretty:SW-TH_XKB_SS-12M11XX
- U4: footprint (none) -> Aliexpress:mini650
Connections:
- net +5V: now also C8.1
- net BAT5v: no longer C8.1
- net D+: no longer J1.A6 (D+), J1.B6 (D+), U2.3 (I/O2)
- net D-: no longer J1.A7 (D-), J1.B7 (D-), U2.1 (I/O1)
- new net: J1.A6 (D+), J1.B6 (D+), U2.3 (I/O2)
- new net: J1.A7 (D-), J1.B7 (D-), U2.1 (I/O1)
Other:
- note added: "Mounting Holes"
- moved on the sheet: J6, J8

Commit message: Pcb fixes
Parts:
- removed D1, D3: ESD9B3.3, Diode_SMD:D_SOD-923, symbol Diode:ESD9B3.3ST5G
Connections:
- net +5V: no longer C8.1
- net BAT5v: now also C8.1
